File: kicad/cell_balancer.sch (KiCad schematic (older format))
At the start: 9 parts, among them U2 BQ29209

Commit message: Updated schematic
Made some error with first rev, the found error are now corrected.
Parts:
- C6, C7, C8, C9: footprint (none) -> Capacitor_SMD:C_0603_1608Metric
- U2: footprint (none) -> outdoor-sense-footprint:BQ29209DRBR
Connections:
- net BAT+ renamed CELL2
Changed lines of the file:
@@
 $Descr A4 11693 8268
 encoding utf-8
-Sheet 4 6
+Sheet 4 7
 Title ""
 Date ""
@@
 Comment4 ""
 $EndDescr
-Text HLabel 3500 2350 0    50   Input ~ 0
-BAT+
 Text HLabel 3450 3650 0    50   Input ~ 0
 BAT-
@@
 F 0 "U2" H 4950 3565 50  0000 C CNN
 F 1 "BQ29209" H 4950 3474 50  0000 C CNN
-F 2 "" H 4800 3000 50  0001 C CNN
+F 2 "outdoor-sense-footprint:BQ29209DRBR" H 4800 3000 50  0001 C CNN
 F 3 "" H 4800 3000 50  0001 C CNN
 	1    4950 3000
@@
 F 0 "C8" H 4592 3546 50  0000 L CNN
 F 1 "0.1uF" H 4592 3455 50  0000 L CNN
-F 2 "" H 4500 3500 50  0001 C CNN
+F 2 "Capacitor_SMD:C_0603_1608Metric" H 4500 3500 50  0001 C CNN
 F 3 "~" H 4500 3500 50  0001 C CNN
 	1    4500 3500
@@
 F 0 "C7" H 4242 3546 50  0000 L CNN
 F 1 "0.1uF" H 4242 3455 50  0000 L CNN
-F 2 "" H 4150 3500 50  0001 C CNN
+F 2 "Capacitor_SMD:C_0603_1608Metric" H 4150 3500 50  0001 C CNN
 F 3 "~" H 4150 3500 50  0001 C CNN
 	1    4150 3500
@@
 F 0 "C6" H 4242 2846 50  0000 L CNN
 F 1 "0.1uF" H 4242 2755 50  0000 L CNN
-F 2 "" H 4150 2800 50  0001 C CNN
+F 2 "Capacitor_SMD:C_0603_1608Metric" H 4150 2800 50  0001 C CNN
 F 3 "~" H 4150 2800 50  0001 C CNN
 	1    4150 2800
@@
 F 0 "C9" H 5692 3546 50  0000 L CNN
 F 1 "0.1uF" H 5692 3455 50  0000 L CNN
-F 2 "" H 5600 3500 50  0001 C CNN
+F 2 "Capacitor_SMD:C_0603_1608Metric" H 5600 3500 50  0001 C CNN
 F 3 "~" H 5600 3500 50  0001 C CNN
 	1    5600 3500
@@
 	5600 3650 5450 3650
 Connection ~ 5450 3650
-Wire Wire Line
-	3500 2350 3700 2350
-Connection ~ 3700 2350
 NoConn ~ 5400 2700
 $EndSCHEMATC
