File: kicad/charge_module.sch (KiCad schematic (older format))
At the start: 19 parts, among them J2 USB_C_Receptacle_USB2.0, U3 BQ25886

Commit message: Updated schematic
Made some error with first rev, the found error are now corrected.
Parts:
- added R5: 0, Resistor_SMD:R_0603_1608Metric, symbol Device:R_Small
- C10, C13: footprint (none) -> Capacitor_SMD:C_0603_1608Metric
- C11, C14: footprint (none) -> Capacitor_SMD:C_0805_2012Metric
- C12: footprint (none) -> Capacitor_SMD:C_1206_3216Metric
- J2: footprint (none) -> connectors:USB_C_JAE_DX07S016JA1R1500
- L2: footprint (none) -> Inductor_SMD:L_Bourns_SRN8040TA
- PG1: renamed from D4; footprint (none) -> Diode_SMD:D_0603_1608Metric
- R19, R20: value R_Small -> 1k
- STAT1: renamed from D3; footprint (none) -> Diode_SMD:D_0603_1608Metric
- TH1: footprint (none) -> Resistor_SMD:R_0603_1608Metric
- U3: footprint (none) -> Package_DFN_QFN:VQFN-24-1EP_4x4mm_P0.5mm_EP2.45x2.45mm_ThermalVias
- renumbered R15 to CC1, R16 to CC2
Connections:
- net VREGN is gone; now on net REGN: R21.2
- net BAT+: now also R19.1, R20.1
- net GND: now also J2.S1 (SHIELD), R5.2
- net ~CE: now also R5.1
- net VBUS: now reaches C10.2, J2.A4 (VBUS), J2.A9 (VBUS), J2.B4 (VBUS), J2.B9 (VBUS), U3.23 (VBUS)
- net ICHGSET: now reaches R17.1, U3.10 (ICHGSET)
- net REGN: now reaches C11.2, U3.11 (REGN)
- net SW: now reaches C13.1, L2.1, U3.17 (SW), U3.18 (SW)
- net PMID: now reaches C12.2, L2.2, U3.21 (PMID), U3.22 (PMID)
- net ILIM: now reaches R18.1, U3.8 (ILIM)
Other:
- note added: "CL21A475KLCLQNC\n"
- note added: "NTCG163JF103HT1"
- note added: "SRN8040TA-1R0Y"
- moved on the sheet: R18
Changed lines of the file:
@@
 $Descr A4 11693 8268
 encoding utf-8
-Sheet 5 6
+Sheet 7 7
 Title ""
 Date ""
@@
 Text HLabel 5450 4250 2    50   Input ~ 0
 BAT-
-Text HLabel 4000 3900 0    50   Input ~ 0
-~CE
 $Comp
 L Powerbank-rescue:USB_C_Receptacle_USB2.0-Connector J?
@@
 F 0 "J2" H 1357 4167 50  0000 C CNN
 F 1 "USB_C_Receptacle_USB2.0" H 1357 4076 50  0000 C CNN
-F 2 "" H 1400 3300 50  0001 C CNN
+F 2 "connectors:USB_C_JAE_DX07S016JA1R1500" H 1400 3300 50  0001 C CNN
 F 3 "https://www.usb.org/sites/default/files/documents/usb_type-c.zip" H 1400 3300 50  0001 C CNN
 	1    1250 3300
@@
 F 0 "U3" H 4500 4265 50  0000 C CNN
 F 1 "BQ25886" H 4500 4174 50  0000 C CNN
-F 2 "" H 4500 3500 50  0001 C CNN
+F 2 "Package_DFN_QFN:VQFN-24-1EP_4x4mm_P0.5mm_EP2.45x2.45mm_ThermalVias" H 4500 3500 50  0001 C CNN
 F 3 "" H 4500 3500 50  0001 C CNN
 	1    4500 3500
@@
 	2100 3500 2100 3700
 $Comp
-L Device:LED_Small D3
+L Device:LED_Small STAT1
 U 1 1 5FBB95AC
 P 5250 2700
-F 0 "D3" H 5250 2935 50  0000 C CNN
+F 0 "STAT1" H 5250 2935 50  0000 C CNN
 F 1 "STAT" H 5250 2844 50  0000 C CNN
-F 2 "" V 5250 2700 50  0001 C CNN
+F 2 "Diode_SMD:D_0603_1608Metric" V 5250 2700 50  0001 C CNN
 F 3 "~" V 5250 2700 50  0001 C CNN
 	1    5250 2700
@@
 $EndComp
 $Comp
-L Device:LED_Small D4
+L Device:LED_Small PG1
 U 1 1 5FBB9A2E
 P 5450 2800
-F 0 "D4" H 5450 3047 50  0000 C CNN
+F 0 "PG1" H 5450 3047 50  0000 C CNN
 F 1 "~PG" H 5450 2949 50  0000 C CNN
-F 2 "" V 5450 2800 50  0001 C CNN
+F 2 "Diode_SMD:D_0603_1608Metric" V 5450 2800 50  0001 C CNN
 F 3 "~" V 5450 2800 50  0001 C CNN
 	1    5450 2800
@@
 P 5700 2700
 F 0 "R19" V 5504 2700 50  0000 C CNN
-F 1 "R_Small" V 5595 2700 50  0000 C CNN
+F 1 "1k" V 5595 2700 50  0000 C CNN
 F 2 "Resistor_SMD:R_0603_1608Metric" H 5700 2700 50  0001 C CNN
 F 3 "~" H 5700 2700 50  0001 C CNN
@@
 P 5950 2800
 F 0 "R20" V 5754 2800 50  0000 C CNN
-F 1 "R_Small" V 5845 2800 50  0000 C CNN
+F 1 "1k" V 5845 2800 50  0000 C CNN
 F 2 "Resistor_SMD:R_0603_1608Metric" H 5950 2800 50  0001 C CNN
 F 3 "~" H 5950 2800 50  0001 C CNN
@@
 L Device:R_Small R18
 U 1 1 5FBBB326
-P 3850 4050
-F 0 "R18" V 3800 4050 50  0000 C CNN
-F 1 "383" V 3850 4050 50  0000 C CNN
-F 2 "Resistor_SMD:R_0603_1608Metric" H 3850 4050 50  0001 C CNN
-F 3 "~" H 3850 4050 50  0001 C CNN
-	1    3850 4050
+P 3650 4050
+F 0 "R18" V 3600 4050 50  0000 C CNN
+F 1 "383" V 3650 4050 50  0000 C CNN
+F 2 "Resistor_SMD:R_0603_1608Metric" H 3650 4050 50  0001 C CNN
+F 3 "~" H 3650 4050 50  0001 C CNN
+	1    3650 4050
 	0    1    1    0
 $EndComp
@@
 	3550 4250 4000 4250
 Wire Wire Line
-	4000 4050 3950 4050
-Wire Wire Line
-	3750 4050 3250 4050
+	4000 4050 3750 4050
+Wire Wire Line
+	3550 4050 3250 4050
 Wire Wire Line
 	3250 4050 3250 4150
@@
 	3250 4150 3250 4250
 $Comp
-L Device:R_Small R15
+L Device:R_Small CC1
 U 1 1 5FBBECAF
 P 2000 2900
-F 0 "R15" V 1804 2900 50  0000 C CNN
+F 0 "CC1" V 1804 2900 50  0000 C CNN
 F 1 "5.1k" V 1895 2900 50  0000 C CNN
 F 2 "Resistor_SMD:R_0603_1608Metric" H 2000 2900 50  0001 C CNN
@@
 $EndComp
 $Comp
-L Device:R_Small R16
+L Device:R_Small CC2
 U 1 1 5FBBEF5D
 P 2200 3000
-F 0 "R16" V 2004 3000 50  0000 C CNN
+F 0 "CC2" V 2004 3000 50  0000 C CNN
 F 1 "5.1k" V 2095 3000 50  0000 C CNN
 F 2 "Resistor_SMD:R_0603_1608Metric" H 2200 3000 50  0001 C CNN
@@
 F 0 "L2" H 3556 2954 50  0000 R CNN
 F 1 "1uH" H 3556 3045 50  0000 R CNN
-F 2 "" H 3600 3000 50  0001 C CNN
+F 2 "Inductor_SMD:L_Bourns_SRN8040TA" H 3600 3000 50  0001 C CNN
 F 3 "~" H 3600 3000 50  0001 C CNN
 	1    3600 3000
@@
 F 0 "C12" V 3679 2900 50  0000 C CNN
 F 1 "10uF" V 3588 2900 50  0000 C CNN
-F 2 "" H 3450 2900 50  0001 C CNN
+F 2 "Capacitor_SMD:C_1206_3216Metric" H 3450 2900 50  0001 C CNN
 F 3 "~" H 3450 2900 50  0001 C CNN
 	1    3450 2900
@@
 F 0 "C13" H 3692 3246 50  0000 L CNN
 F 1 "47nF" H 3692 3155 50  0000 L CNN
-F 2 "" H 3600 3200 50  0001 C CNN
+F 2 "Capacitor_SMD:C_0603_1608Metric" H 3600 3200 50  0001 C CNN
 F 3 "~" H 3600 3200 50  0001 C CNN
 	1    3600 3200
@@
 F 0 "C11" V 3429 3400 50  0000 C CNN
 F 1 "4.7uF" V 3338 3400 50  0000 C CNN
-F 2 "" H 3200 3400 50  0001 C CNN
+F 2 "Capacitor_SMD:C_0805_2012Metric" H 3200 3400 50  0001 C CNN
 F 3 "~" H 3200 3400 50  0001 C CNN
 	1    3200 3400
@@
 Wire Wire Line
 	4000 3800 3250 3800
-Wire Wire Line
-	3250 3800 3250 4050
 Connection ~ 3250 4050
 Text Notes 3400 4550 0    50   ~ 0
@@
 F 0 "C10" H 2508 2854 50  0000 R CNN
 F 1 "1uF" H 2508 2945 50  0000 R CNN
-F 2 "" H 2600 2900 50  0001 C CNN
+F 2 "Capacitor_SMD:C_0603_1608Metric" H 2600 2900 50  0001 C CNN
 F 3 "~" H 2600 2900 50  0001 C CNN
 	1    2600 2900
@@
 F 0 "TH1" H 6755 3546 50  0000 L CNN
 F 1 "10k" H 6755 3455 50  0000 L CNN
-F 2 "" H 6650 3500 50  0001 C CNN
+F 2 "Resistor_SMD:R_0603_1608Metric" H 6650 3500 50  0001 C CNN
 F 3 "~" H 6650 3500 50  0001 C CNN
 	1    6650 3500
@@
 Wire Wire Line
 	6050 3000 6050 2950
-Text Label 6050 2950 0    50   ~ 0
-VREGN
 Wire Wire Line
 	5000 3300 6050 3300
@@
 F 0 "C14" H 5842 3096 50  0000 L CNN
 F 1 "4.7uF" H 5842 3005 50  0000 L CNN
-F 2 "" H 5750 3050 50  0001 C CNN
+F 2 "Capacitor_SMD:C_0805_2012Metric" H 5750 3050 50  0001 C CNN
 F 3 "~" H 5750 3050 50  0001 C CNN
 	1    5750 3050
@@
 Wire Wire Line
 	5750 2900 5750 2950
+Text Label 3450 3400 0    50   ~ 0
+REGN
+Text Label 6050 2950 0    50   ~ 0
+REGN
+Text HLabel 6150 2700 2    50   Input ~ 0
+BAT+
+Text Notes 6950 3550 0    50   ~ 0
+NTCG163JF103HT1
+Text Notes 2850 3600 0    50   ~ 0
+CL21A475KLCLQNC\n
+Text Notes 2850 3050 0    50   ~ 0
+SRN8040TA-1R0Y
+Text Label 3800 2900 0    50   ~ 0
+PMID
+Text Label 3850 3100 0    50   ~ 0
+SW
+Text Label 3800 4050 0    50   ~ 0
+ILIM
+Text Label 3650 4250 0    50   ~ 0
+ICHGSET
+$Comp
+L power:GND #PWR0132
+U 1 1 5FC8B6A1
+P 950 4200
+F 0 "#PWR0132" H 950 3950 50  0001 C CNN
+F 1 "GND" H 955 4027 50  0000 C CNN
+F 2 "" H 950 4200 50  0001 C CNN
+F 3 "" H 950 4200 50  0001 C CNN
+	1    950  4200
+	1    0    0    -1
+$EndComp
+Text Label 3800 3900 0    50   ~ 0
+~CE
+Wire Wire Line
+	4000 3900 3800 3900
+Wire Wire Line
+	3250 3800 3250 3900
+$Comp
+L Device:R_Small R5
+U 1 1 5FC76A50
+P 3700 3900
+F 0 "R5" V 3650 3900 50  0000 C CNN
+F 1 "0" V 3700 3900 50  0000 C CNN
+F 2 "Resistor_SMD:R_0603_1608Metric" H 3700 3900 50  0001 C CNN
+F 3 "~" H 3700 3900 50  0001 C CNN
+	1    3700 3900
+	0    1    1    0
+$EndComp
+Wire Wire Line
+	3600 3900 3250 3900
+Connection ~ 3250 3900
+Wire Wire Line
+	3250 3900 3250 4050
+Text Label 2600 2700 0    50   ~ 0
+VBUS
 $EndSCHEMATC
